Commit message: creamos nuevo launcher para meter al rover en el mundo proporcionado y cambios a urdf para que todo funcione

File: urdf/arm/arm.urdf.xacro (robot description, xacro)
@@ -107,13 +107,19 @@
       <axis xyz="0 0 1"/>
     </joint>
-    <link name="Cylinder_link"/>
+    <link name="Cylinder_link">
+      <inertial>
+        <mass value="0.01"/>
+        <origin xyz="0 0 0" rpy="0 0 0"/>
+        <inertia ixx="0.0001" ixy="0" ixz="0" iyy="0.0001" iyz="0" izz="0.0001"/>
+      </inertial>
+    </link>
     <joint name="Cylinder_vertical_joint" type="prismatic">
       <limit lower="-1.5" upper="1.1" effort="10.0" velocity="1.0"/>
       <origin xyz="0 0 -1.39867" rpy="0 0 0"/>
       <parent link="Cylinder_link"/>
-      <child link="Cylinder_link.001"/>
-      <axis xyz="0 0 1"/>
-    </joint>
-    <link name="Cylinder_link.001">
+      <child link="cylinder_link_001"/>
+      <axis xyz="0 0 1"/>
+    </joint>
+    <link name="cylinder_link_001">
       <inertial>
         <inertia ixx="0.9401" ixy="0.0" ixz="0.0" iyy="0.9401" iyz="0.0" izz="0.0125"/>
@@ -135,5 +141,5 @@
     <joint name="base_gripper_joint" type="fixed">
       <origin xyz="0 0 -1.57568" rpy="0 0 0"/>
-      <parent link="Cylinder_link.001"/>
+      <parent link="cylinder_link_001"/>
       <child link="base_gripper_link"/>
     </joint>

File: urdf/sensors/camera.urdf.xacro (robot description, xacro)
@@ -16,4 +16,9 @@
         </material>
       </visual>
+      <inertial>
+        <mass value="0.01"/>
+        <origin xyz="0 0 0" rpy="0 0 0"/>
+        <inertia ixx="0.0001" ixy="0" ixz="0" iyy="0.0001" iyz="0" izz="0.0001"/>
+      </inertial>
     </link>
     <gazebo reference="${frame_prefix}_camera_frame">

File: urdf/sensors/imu.urdf.xacro (robot description, xacro)
@@ -3,4 +3,9 @@
   <xacro:macro name="imu_sensor" params="parent">
     <link name="imu_link"/>
+      <inertial>
+        <mass value="0.01"/>
+        <origin xyz="0 0 0" rpy="0 0 0"/>
+        <inertia ixx="0.0001" ixy="0" ixz="0" iyy="0.0001" iyz="0" izz="0.0001"/>
+      </inertial>
     <joint name="imu_link_jonit" type="fixed">
       <parent link="${parent}"/>

Commit message: Añado limites de acceleracion, ya puedo planificar movimientos con el scara

File: urdf/arm/arm.urdf.xacro (robot description, xacro)
@@ -25,6 +25,7 @@
       </visual>
     </link>
+    <!-- Articulación 1: Rotación Hombro -->
     <joint name="scara_arm_1_link_joint" type="revolute">
-      <limit lower="-2.27" upper="4.17" effort="1000.0" velocity="10.0"/>
+      <limit lower="-2.27" upper="4.17" effort="1000.0" velocity="10.0" acceleration="5.0"/>
       <origin xyz="0.0 0.0 0.52512" rpy="0 0 0"/>
       <parent link="scara_base_link"/>
@@ -73,6 +74,7 @@
       </visual>
     </link>
+    <!-- Articulación 3: Rotación Codo -->
     <joint name="scara_arm_3_link_joint" type="revolute">
-      <limit lower="-1.2" upper="4.3" effort="1000.0" velocity="10.0"/>
+      <limit lower="-1.2" upper="4.3" effort="1000.0" velocity="10.0" acceleration="5.0"/>
       <origin xyz="0.0 0.64991 0.2" rpy="0 0 0"/>
       <parent link="scara_arm_2_link"/>
@@ -100,6 +102,7 @@
       </visual>
     </link>
+    <!-- Articulación 4: Rotación Muñeca -->
     <joint name="Cylinder_rotational_joint" type="revolute">
-      <limit lower="-3.14" upper="3.14" effort="1000.0" velocity="10.0"/>
+      <limit lower="-3.14" upper="3.14" effort="1000.0" velocity="10.0" acceleration="5.0"/>
       <origin xyz="1.26955 0 1.51933" rpy="0 0 0.7854"/>
       <parent link="scara_arm_3_link"/>
@@ -114,6 +117,7 @@
       </inertial>
     </link>
+    <!-- Articulación 5: Movimiento Vertical (Prismático) -->
     <joint name="Cylinder_vertical_joint" type="prismatic">
-      <limit lower="-1.5" upper="1.1" effort="1000.0" velocity="10.0"/>
+      <limit lower="-1.5" upper="1.1" effort="1000.0" velocity="10.0" acceleration="2.0"/>
       <origin xyz="0 0 -1.39867" rpy="0 0 0"/>
       <parent link="Cylinder_link"/>
@@ -162,6 +166,7 @@
       </visual>
     </link>
+    <!-- Articulación 6: Dedo Izquierdo -->
     <joint name="left_grip_joint" type="prismatic">
-      <limit lower="0.0" upper="0.07" effort="1000.0" velocity="10.0"/>
+      <limit lower="0.0" upper="0.07" effort="1000.0" velocity="10.0" acceleration="2.0"/>
       <origin xyz="0 -0.325 -0.17515" rpy="0 0 0"/>
       <parent link="base_gripper_link"/>
@@ -187,6 +192,7 @@
       </visual>
     </link>
+    <!-- Articulación 7: Dedo Derecho -->
     <joint name="right_grip_joint" type="prismatic">
-      <limit lower="-0.07" upper="0.0" effort="1000.0" velocity="10.0"/>
+      <limit lower="-0.07" upper="0.0" effort="1000.0" velocity="10.0" acceleration="2.0"/>
       <origin xyz="0 0.3248 -0.17515" rpy="0 0 0"/>
       <parent link="base_gripper_link"/>
