Commit message: modelo robot usando xacro

File: robots/robot.urdf.xacro (robot description, xacro)
@@ -6,4 +6,6 @@
   <xacro:include filename="$(find rover_description)/urdf/wheels/axis.urdf.xacro"/>
   <xacro:include filename="$(find rover_description)/urdf/arm/arm.urdf.xacro"/>
+  <xacro:include filename="$(find rover_description)/urdf/sensors/imu.urdf.xacro"/>
+  <xacro:include filename="$(find rover_description)/urdf/sensors/camera.urdf.xacro"/>
   <xacro:property name="Front_wheel_offset_x" value="1.6"/>
   <xacro:property name="Middle_wheel_offset_x" value="-0.1"/>
@@ -61,3 +63,21 @@
     <origin xyz="0.71003 -0.01046 0.71815" rpy="0 0 0"/>
   </xacro:scara_arm>
+  <!-- SENSORS -->
+  <xacro:imu_sensor parent="base_link"/>
+  <xacro:sensor_camera
+    frame_prefix="front"
+    parent="base_link"
+    horizontal_fov="90"
+    video_width="640"
+    video_height="480">
+    <origin xyz="1.05 0 0.5" rpy="0 0 0"/>
+  </xacro:sensor_camera>
+  <xacro:sensor_camera
+      frame_prefix="gripper"
+      parent="base_gripper_link"
+      horizontal_fov="60"
+      video_width="640"
+      video_height="480">
+    <origin xyz="0 0 -0.05" rpy="0 0 0"/>
+  </xacro:sensor_camera>
 </robot>

Commit message: Hay error en alguna parte, no se me visauliza bien en rviz ahora

File: robots/robot.urdf.xacro (robot description, xacro)
@@ -3,4 +3,5 @@
 <robot name="robot" xmlns:xacro="http://wiki.ros.org/xacro">
   <xacro:include filename="$(find rover_description)/urdf/base/rover_base.urdf.xacro"/>
+  <xacro:include filename="$(find rover_description)/urdf/base/envase.urdf.xacro"/>
   <xacro:include filename="$(find rover_description)/urdf/wheels/rover_wheel.urdf.xacro"/>
   <xacro:include filename="$(find rover_description)/urdf/wheels/axis.urdf.xacro"/>
@@ -8,4 +9,5 @@
   <xacro:include filename="$(find rover_description)/urdf/sensors/imu.urdf.xacro"/>
   <xacro:include filename="$(find rover_description)/urdf/sensors/camera.urdf.xacro"/>
+  <xacro:include filename="$(find rover_description)/urdf/utils/arm_plugins.urdf.xacro" />
   <xacro:property name="Front_wheel_offset_x" value="1.6"/>
   <xacro:property name="Middle_wheel_offset_x" value="-0.1"/>
@@ -14,5 +16,4 @@
   <xacro:property name="Axis_offset_z" value="-1.05"/>
   <xacro:property name="Axis_to_wheel_offset_y" value="0.2"/>
-  <xacro:include filename="$(find rover_description)/urdf/utils/envase.urdf.xacro"/>
   <!-- BASE -->
   <xacro:robot_base/>
@@ -81,3 +82,4 @@
     <origin xyz="0 0 -0.05" rpy="0 0 0"/>
   </xacro:sensor_camera>
+  <!-- Controlador Gazebo ros2  -->
 </robot>

File: urdf/arm/arm.urdf.xacro (robot description, xacro)
@@ -129,11 +129,11 @@
       <collision>
         <geometry>
-          <mesh filename="package://rover_description/meshes/dae/Cylinder.002.dae" scale="0.1 0.1 1.5"/>
-        </geometry>
-      </collision>
-      <visual>
-        <material name="Material.007"/>
-        <geometry>
-          <mesh filename="package://rover_description/meshes/dae/Cylinder.002.dae" scale="0.1 0.1 1.5"/>
+          <mesh filename="file://$(find rover_description)/meshes/dae/Cylinder.002.dae" scale="0.1 0.1 1.5"/>
+        </geometry>
+      </collision>
+      <visual>
+        <material name="Material.007"/>
+        <geometry>
+          <mesh filename="file://$(find rover_description)/meshes/dae/Cylinder.002.dae" scale="0.1 0.1 1.5"/>
         </geometry>
       </visual>

File: urdf/base/envase.urdf.xacro (robot description, xacro)
@@ -52,5 +52,5 @@
         <origin rpy="0.00000 0.00000 0.00000" xyz="0.00000 0.00471 0.00000"/>
         <geometry>
-          <mesh filename="package://rover_description/meshes/dae/Cube.020.dae" scale="0.97000 0.35000 0.05000"/>
+          <mesh filename="file://$(find rover_description)/meshes/dae/Cube.020.dae" scale="0.97000 0.35000 0.05000"/>
         </geometry>
       </visual>

File: urdf/base/rover_base.urdf.xacro (robot description, xacro)
@@ -41,5 +41,5 @@
         <origin rpy="0.00000 -0.78540 0.00000" xyz="0.00000 0.00000 0.00000"/>
         <geometry>
-          <mesh filename="package://rover_description/meshes/dae/Cube.011.dae" scale="0.05000 0.05250 0.05000"/>
+          <mesh filename="file://$(find rover_description)/meshes/dae/Cube.011.dae" scale="0.05000 0.05250 0.05000"/>
         </geometry>
       </visual>

File: urdf/wheels/rover_wheel.urdf.xacro (robot description, xacro)
@@ -12,5 +12,5 @@
         <origin rpy="-1.57080 0.00000 0.00000" xyz="0.00000 0.00000 0.00000"/>
         <geometry>
-          <mesh filename="package://rover_description/meshes/dae/${mesh_file}" scale="0.05000 0.05000 0.12500"/>
+          <mesh filename="file://$(find rover_description)/meshes/dae/${mesh_file}" scale="0.05000 0.05000 0.12500"/>
         </geometry>
       </visual>
@@ -18,5 +18,5 @@
         <origin rpy="-1.57080 0.00000 0.00000" xyz="0.00000 0.00000 0.00000"/>
         <geometry>
-          <mesh filename="package://rover_description/meshes/dae/${mesh_file}" scale="0.05000 0.05000 0.12500"/>
+          <mesh filename="file://$(find rover_description)/meshes/dae/${mesh_file}" scale="0.05000 0.05000 0.12500"/>
         </geometry>
       </collision>

Commit message: se me lanza todo sin errores

File: robots/robot.urdf.xacro (robot description, xacro)
@@ -10,4 +10,5 @@
   <xacro:include filename="$(find rover_description)/urdf/sensors/camera.urdf.xacro"/>
   <xacro:include filename="$(find rover_description)/urdf/utils/arm_plugins.urdf.xacro" />
+  <xacro:include filename="$(find rover_description)/urdf/utils/ros2_control.urdf.xacro" />
   <xacro:property name="Front_wheel_offset_x" value="1.6"/>
   <xacro:property name="Middle_wheel_offset_x" value="-0.1"/>
@@ -83,3 +84,7 @@
   </xacro:sensor_camera>
   <!-- Controlador Gazebo ros2  -->
+  <xacro:arg name="config_controllers" default="$(find rover_description)/config/rover_controllers.yaml"/>
+  <xacro:arg name="update_rate" default="20"/>
+  <!-- Esta es la llamada que activa todo el sistema de control -->
+  <xacro:ros2_control/>
 </robot>

File: urdf/arm/arm.urdf.xacro (robot description, xacro)
@@ -26,5 +26,5 @@
     </link>
     <joint name="scara_arm_1_link_joint" type="revolute">
-      <limit lower="-2.27" upper="4.17" effort="10.0" velocity="1.0"/>
+      <limit lower="-2.27" upper="4.17" effort="1000.0" velocity="10.0"/>
       <origin xyz="0.0 0.0 0.52512" rpy="0 0 0"/>
       <parent link="scara_base_link"/>
@@ -74,5 +74,5 @@
     </link>
     <joint name="scara_arm_3_link_joint" type="revolute">
-      <limit lower="-1.2" upper="4.3" effort="10.0" velocity="1.0"/>
+      <limit lower="-1.2" upper="4.3" effort="1000.0" velocity="10.0"/>
       <origin xyz="0.0 0.64991 0.2" rpy="0 0 0"/>
       <parent link="scara_arm_2_link"/>
@@ -101,5 +101,5 @@
     </link>
     <joint name="Cylinder_rotational_joint" type="revolute">
-      <limit lower="-3.14" upper="3.14" effort="10.0" velocity="1.0"/>
+      <limit lower="-3.14" upper="3.14" effort="1000.0" velocity="10.0"/>
       <origin xyz="1.26955 0 1.51933" rpy="0 0 0.7854"/>
       <parent link="scara_arm_3_link"/>
@@ -115,5 +115,5 @@
     </link>
     <joint name="Cylinder_vertical_joint" type="prismatic">
-      <limit lower="-1.5" upper="1.1" effort="10.0" velocity="1.0"/>
+      <limit lower="-1.5" upper="1.1" effort="1000.0" velocity="10.0"/>
       <origin xyz="0 0 -1.39867" rpy="0 0 0"/>
       <parent link="Cylinder_link"/>
@@ -163,5 +163,5 @@
     </link>
     <joint name="left_grip_joint" type="prismatic">
-      <limit lower="0.0" upper="0.07" effort="10.0" velocity="1.0"/>
+      <limit lower="0.0" upper="0.07" effort="1000.0" velocity="10.0"/>
       <origin xyz="0 -0.325 -0.17515" rpy="0 0 0"/>
       <parent link="base_gripper_link"/>
@@ -188,5 +188,5 @@
     </link>
     <joint name="right_grip_joint" type="prismatic">
-      <limit lower="-0.07" upper="0.0" effort="10.0" velocity="1.0"/>
+      <limit lower="-0.07" upper="0.0" effort="1000.0" velocity="10.0"/>
       <origin xyz="0 0.3248 -0.17515" rpy="0 0 0"/>
       <parent link="base_gripper_link"/>

File: urdf/base/rover_base.urdf.xacro (robot description, xacro)
@@ -2,5 +2,7 @@
 <robot xmlns:xacro="http://wiki.ros.org/xacro">
   <xacro:macro name="robot_base">
+    <!-- Enlace en el suelo: fíjate que se cierra con /> al final -->
     <link name="base_footprint"/>
+    <!-- Unión fija entre el suelo y el chasis -->
     <joint name="base_footprint_joint" type="fixed">
       <parent link="base_footprint"/>
@@ -10,8 +12,8 @@
     <link name="base_link">
       <collision name="chasis_collision">
-      <origin rpy="0.00000 0.00000 0.00000" xyz="0.05491 -0.59562 -0.76184"/>
-      <geometry>
-        <box size="3.20000 0.10000 0.90000"/>
-      </geometry>
+        <origin rpy="0.00000 0.00000 0.00000" xyz="0.05491 -0.59562 -0.76184"/>
+        <geometry>
+          <box size="3.20000 0.10000 0.90000"/>
+        </geometry>
       </collision>
       <collision name="chasis_collision.001">

File: urdf/utils/ros2_control.urdf.xacro (robot description, xacro)
@@ -1,10 +1,10 @@
 <?xml version="1.0"?>
 <robot xmlns:xacro="http://www.ros.org/wiki/xacro">
-  <xacro:macro name="rover_diff_drive">
+  <xacro:macro name="ros2_control">
     <!-- 1. EL PLUGIN PRINCIPAL (El que carga ros2_control en Gazebo) -->
     <!-- IMPORTANTE: Solo puede haber uno de estos en todo el robot. Si ya lo tienes en el brazo, no lo repitas -->
     <gazebo>
       <plugin filename="libgz_ros2_control-system.so" name="gz_ros2_control::GazeboSimROS2ControlPlugin">
-        <parameters>$(find rover_moveit_config)/config/ros2_controllers.yaml</parameters>
+        <parameters>$(find robot_moveit_config)/config/ros2_controllers.yaml</parameters>
       </plugin>
     </gazebo>

Commit message: Añado etiquetas en las wheels para poder teleoperar el rover

File: robots/robot.urdf.xacro (robot description, xacro)
@@ -61,4 +61,12 @@
     <origin xyz="0 -${Axis_to_wheel_offset_y} 0" rpy="${pi/2} 0 0"/>
   </xacro:rover_wheel>
+  <!-- Fricción para ruedas izquierdas -->
+  <gazebo reference="front_left_wheel_link"><mu1>0.1</mu1><mu2>0.1</mu2></gazebo>
+  <gazebo reference="middle_left_wheel_link"><mu1>1.0</mu1><mu2>1.0</mu2></gazebo>
+  <gazebo reference="back_left_wheel_link"><mu1>0.1</mu1><mu2>0.1</mu2></gazebo>
+  <!-- Fricción para ruedas derechas -->
+  <gazebo reference="front_right_wheel_link"><mu1>0.1</mu1><mu2>0.1</mu2></gazebo>
+  <gazebo reference="middle_right_wheel_link"><mu1>1.0</mu1><mu2>1.0</mu2></gazebo>
+  <gazebo reference="back_right_wheel_link"><mu1>0.1</mu1><mu2>0.1</mu2></gazebo>
   <!-- ARM -->
   <xacro:scara_arm parent="base_link">

File: urdf/wheels/rover_wheel.urdf.xacro (robot description, xacro)
@@ -6,5 +6,5 @@
       <parent link="${parent}"/>
       <child link="${prefix}_wheel_link"/>
-      <axis xyz="0 0 1"/> <limit effort="10.0" velocity="1.0"/>
+      <axis xyz="0 0 -1"/> <limit effort="200.0" velocity="10.0"/>
     </joint>
     <link name="${prefix}_wheel_link">
@@ -27,4 +27,13 @@
       </inertial>
     </link>
+    <gazebo reference="${prefix}_wheel_link">
+      <mu1>1.0</mu1>
+      <mu2>0.1</mu2>
+      <kp>1000000.0</kp>
+      <kd>10.0</kd>
+      <minDepth>0.001</minDepth>
+      <maxVel>0.1</maxVel>
+      <fdir1>1 0 0</fdir1>
+    </gazebo>
   </xacro:macro>
 </robot>

Commit message: ajustes en las ruedas para los giros, camara gripper mirando hacia abajo, imu publicandose

File: robots/robot.urdf.xacro (robot description, xacro)
@@ -74,5 +74,8 @@
   </xacro:scara_arm>
   <!-- SENSORS -->
-  <xacro:imu_sensor parent="base_link"/>
+  <xacro:sensor_imu prefix="imu" parent="base_link">
+    <!-- Aquí defines la posición física de la IMU respecto al parent -->
+    <origin xyz="1.0 0.0 0.5" rpy="0 0 0"/>
+  </xacro:sensor_imu>
   <xacro:sensor_camera
     frame_prefix="front"
@@ -89,5 +92,5 @@
       video_width="640"
       video_height="480">
-    <origin xyz="0 0 -0.05" rpy="0 0 0"/>
+    <origin xyz="0 0 -0.05" rpy="0 1.5708 0"/>
   </xacro:sensor_camera>
   <!-- Controlador Gazebo ros2  -->

File: urdf/base/rover_base.urdf.xacro (robot description, xacro)
@@ -38,5 +38,5 @@
         <inertia ixx="155.51313" ixy="0.29579" ixz="-3.95758" iyy="456.61426" iyz="-0.74765" izz="404.59665"/>
         <origin rpy="0.00000 0.00000 0.00000" xyz="0.07609 -0.02047 -0.07797"/>
-        <mass value="500.00000"/>
+        <mass value="100.00000"/>
       </inertial>
       <visual name="chasis">

File: urdf/sensors/imu.urdf.xacro (robot description, xacro)
@@ -1,21 +1,37 @@
 <?xml version="1.0"?>
-<robot xmlns:xacro="http://wiki.ros.org/xacro">
-  <xacro:macro name="imu_sensor" params="parent">
-    <link name="imu_link"/>
+<robot name="imu_sensor" xmlns:xacro="http://wiki.ros.org/xacro">
+  <!-- ######### IMU ######### -->
+  <xacro:macro name="sensor_imu" params="prefix ns:='' topic:='imu/data' parent *origin">
+    <joint name="${prefix}_joint" type="fixed">
+      <xacro:insert_block name="origin" />
+      <parent link="${parent}"/>
+      <child link="${prefix}_link"/>
+    </joint>
+    <link name="${prefix}_link">
       <inertial>
-        <mass value="0.01"/>
-        <origin xyz="0 0 0" rpy="0 0 0"/>
+        <origin xyz="0.0 0.0 0.01" rpy="0 0 0" />
+        <mass value="0.005" />
         <inertia ixx="0.0001" ixy="0" ixz="0" iyy="0.0001" iyz="0" izz="0.0001"/>
       </inertial>
-    <joint name="imu_link_jonit" type="fixed">
-      <parent link="${parent}"/>
-      <child link="imu_link"/>
-      <origin xyz="1 0 0" rpy="0 0 0"/>
-    </joint>
-    <gazebo reference="imu_link">
-      <sensor name="imu_sensor" type="imu">
-      <always_on>1</always_on>
-      <update_rate>30</update_rate>
-      <topic>imu</topic>
+      <visual>
+        <origin rpy="0 0 0" xyz="0 0 0" />
+        <geometry>
+          <box size="0.001 0.001 0.001" />
+        </geometry>
+      </visual>
+    </link>
+    <gazebo reference="${prefix}_link">
+      <sensor name="${prefix}_sensor" type="imu">
+        <always_on>1</always_on>
+        <update_rate>30</update_rate>
+        <visualize>true</visualize>
+        <topic>${topic}</topic>
+        <!-- ESTO ES LO QUE TE FALTA: El puente con ROS 2 -->
+        <plugin name="${prefix}_imu_plugin" filename="libgazebo_ros_imu_sensor.so">
+          <ros>
+            <namespace>${ns}</namespace>
+            <remapping>~/out:=${topic}</remapping>
+          </ros>
+        </plugin>
       </sensor>
     </gazebo>

File: urdf/wheels/rover_wheel.urdf.xacro (robot description, xacro)
@@ -6,5 +6,5 @@
       <parent link="${parent}"/>
       <child link="${prefix}_wheel_link"/>
-      <axis xyz="0 0 -1"/> <limit effort="200.0" velocity="10.0"/>
+      <axis xyz="0 0 -1"/> <limit effort="500.0" velocity="10.0"/>
     </joint>
     <link name="${prefix}_wheel_link">
@@ -28,8 +28,8 @@
     </link>
     <gazebo reference="${prefix}_wheel_link">
-      <mu1>1.0</mu1>
-      <mu2>0.1</mu2>
+      <mu1>0.01</mu1>
+      <mu2>0.01</mu2>
       <kp>1000000.0</kp>
-      <kd>10.0</kd>
+      <kd>100.0</kd>
       <minDepth>0.001</minDepth>
       <maxVel>0.1</maxVel>
